File: PCB/3CIE.kicad_pcb (KiCad board)
At the start: 4 copper layers, 108.7 x 56 mm, 58 parts, among them J1 Bus_PCI_Express_x1, J2 Bus_PCI_Express_x1, J3 Bus_PCI_Express_x1, J4 Bus_PCI_Express_Mini, J5 Bus_PCI_Express_Mini, J6 Bus_PCI_Express_Mini

Commit message: fix logo placement
Parts:
- moved G*** 1.85 mm to (53.0, -10.3)
Other:
- board text removed: "A project by nuccinc.org"

Commit message: push production files / fix board fill
Parts:
- J4, J5, J6: footprint PCIE-Adapter:BUS_PCI_Express_Mini_Half -> 3CIE:BUS_PCI_Express_Mini_Half
Connections:
- J4 pad : (no net) -> GND
- J4 pad 1: WAKE1 -> (no net)
- J5 pad : (no net) -> GND
- J6 pad : (no net) -> GND
Routing:
- net +3V3: track 104.6 -> 111.9 mm
- net GND: vias 341 -> 348
Other:
- board text added: "Differential Pairs: 85OHM (JLC04161H-7628)"
