File: PCB/3CIE.kicad_sch (KiCad schematic)
At the start: 75 parts, among them J1 Bus_PCI_Express_x1, J2 Bus_PCI_Express_x1, J3 Bus_PCI_Express_x1, J4 Bus_PCI_Express_Mini, J5 Bus_PCI_Express_Mini, J6 Bus_PCI_Express_Mini

Commit message: push production files / fix board fill
Parts:
- C1, C11, C13, C15, C16, C17, C18, C2, C4, C6, C7, C9: JLCPCB Part# (none) -> C22435929
- C10, C5, C8: value 47uF -> 22uF; JLCPCB Part# (none) -> C105226
- C12, C14, C3: JLCPCB Part# (none) -> C315248
- D1, D2, D3: JLCPCB Part# (none) -> C122862
- D10, D11, D12, D13, D14, D15, D7, D8, D9: JLCPCB Part# (none) -> C30584803
- J1, J2, J3: now not fitted
- J4, J5, J6: JLCPCB Part# (none) -> C920235
- R1, R13, R14, R19, R2, R20, R21, R7, R8: JLCPCB Part# (none) -> C60490
- R10, R11, R12, R16, R17, R18, R4, R5, R6: JLCPCB Part# (none) -> C105875
- R15, R3, R9: JLCPCB Part# (none) -> C106232
- TP1, TP10, TP11, TP12, TP13, TP14, TP15, TP16, TP17, TP18, TP2, TP3, TP4, TP5, TP6, TP7, TP8, TP9: now not fitted; now left out of the parts list
